Commit message: ydlidar package: occurrences of /laser_frame replaced by /base_scan

File: Chapter9_GoPiGo3_SLAM/ydlidar/urdf/ydlidar.urdf (robot description, URDF)
Before this commit: robot ydlidar, 2 links, 1 joints
Links:
- removed link laser_frame
- added link base_scan, mass 0.25482
Joints:
- joint laser_joint: child laser_frame -> base_scan
